File: IL2237_PCB.kicad_sch (KiCad schematic)
At the start: 17 parts, among them J1 OLED_Display, SW1 SW_Push, SW2 SW_Push, SW3 SW_Push, U1 XIAO-ESP32-C6-SMD

Commit message: finished routing
Parts:
- added H1, H2, H3, H4: MountingHole, MountingHole:MountingHole_2.5mm_Pad, symbol Mechanical:MountingHole
- C1, C2, C3: footprint (none) -> Capacitor_THT:C_Disc_D5.0mm_W2.5mm_P2.50mm
- D1, D2, D3: footprint (none) -> LED_THT:LED_D5.0mm
- J1: footprint (none) -> Connector_PinHeader_2.54mm:PinHeader_1x04_P2.54mm_Vertical
- R1, R2, R3, R4, R5, R6: footprint (none) -> Resistor_THT:R_Axial_DIN0207_L6.3mm_D2.5mm_P7.62mm_Horizontal
- SW1, SW2, SW3: footprint (none) -> Button_Switch_THT:SW_PUSH_6mm
Connections:
- net +3.3V: now also U1.22 (3V3); no longer U1.31 (3V3)
- net GND: now also U1.18 (GND), U1.24 (GND); no longer U1.27 (GND), U1.33 (GND)
- no-connect marks 0 -> 12
